File: 2027_Rev1_BLJoCo_Hardware/2027_BLJoCo_Board/2027_BLJoCo_Board.kicad_pcb (KiCad board)
At the start: 0 parts

Commit message: Footprints assigned
Footprints assigned and board almost complete.
Parts:
- added C10: 100nF, Capacitor_SMD:C_0603_1608Metric_Pad1.08x0.95mm_HandSolder, F.Cu at (100.6, 65.8)
- added C2: 100nF, Capacitor_SMD:C_0603_1608Metric_Pad1.08x0.95mm_HandSolder, F.Cu at (100.6, 50.7)
- added C20: 4.7uF, Capacitor_SMD:C_0603_1608Metric_Pad1.08x0.95mm_HandSolder, F.Cu at (105.0, 50.7)
- added C21: 100nF, Capacitor_SMD:C_0603_1608Metric_Pad1.08x0.95mm_HandSolder, F.Cu at (105.0, 53.3)
- added C22: 10nF, Capacitor_SMD:C_0603_1608Metric_Pad1.08x0.95mm_HandSolder, F.Cu at (105.0, 55.8)
- added C23: 1uF, Capacitor_SMD:C_0603_1608Metric_Pad1.08x0.95mm_HandSolder, F.Cu at (105.0, 58.3)
- added C24: 4.7uF, Capacitor_SMD:C_0603_1608Metric_Pad1.08x0.95mm_HandSolder, F.Cu at (105.0, 60.8)
- added C25: 100nF, Capacitor_SMD:C_0603_1608Metric_Pad1.08x0.95mm_HandSolder, F.Cu at (105.0, 63.3)
- added C26: 100nF, Capacitor_SMD:C_0603_1608Metric_Pad1.08x0.95mm_HandSolder, F.Cu at (105.0, 65.8)
- added C27: 100nF, Capacitor_SMD:C_0603_1608Metric_Pad1.08x0.95mm_HandSolder, F.Cu at (109.3, 50.7)
- added C4: 100nF, Capacitor_SMD:C_0603_1608Metric_Pad1.08x0.95mm_HandSolder, F.Cu at (210.2, 118.3)
- added C5: 22uF, Capacitor_SMD:C_0603_1608Metric_Pad1.08x0.95mm_HandSolder, F.Cu at (207.4, 124.3)
- added C6: 10uF, Capacitor_SMD:C_0603_1608Metric_Pad1.08x0.95mm_HandSolder, F.Cu at (204.7, 115.0)
- added C7: 100nF, Capacitor_SMD:C_0603_1608Metric_Pad1.08x0.95mm_HandSolder, F.Cu at (100.6, 60.8)
- added C8: 22uF, Capacitor_SMD:C_0603_1608Metric_Pad1.08x0.95mm_HandSolder, F.Cu at (207.4, 126.3)
- added C9: 100uf, Capacitor_THT:CP_Radial_D8.0mm_P3.50mm, F.Cu at (204.4, 100.9)
- added D1: MMSZ4685-TP, Diode_SMD:D_SOD-523, F.Cu at (210.1, 126.8)
- added D2: GREEN, LED_SMD:LED_0603_1608Metric_Pad1.05x0.95mm_HandSolder, F.Cu at (133.7, 50.8)
- added D3: GREEN, LED_SMD:LED_0603_1608Metric_Pad1.05x0.95mm_HandSolder, F.Cu at (133.7, 53.4)
- added D4: D_TVS, Diode_SMD:D_0603_1608Metric_Pad1.05x0.95mm_HandSolder, F.Cu at (133.7, 56.0)
- added D5: D_TVS, Diode_SMD:D_0603_1608Metric_Pad1.05x0.95mm_HandSolder, F.Cu at (133.7, 58.6)
- added D6: MMSZ5240BT1G, Diode_SMD:D_SOD-123, F.Cu at (202.6, 110.2)
- added H1: MountingHole_Pad, MountingHole:MountingHole_3.2mm_M3_Pad, F.Cu at (180.6, 83.8)
- added H2: MountingHole_Pad, MountingHole:MountingHole_3.2mm_M3_Pad, F.Cu at (225.3, 83.8)
- added J1: Conn_01x03, Connector_Wire:SolderWire-0.5sqmm_1x03_P4.6mm_D0.9mm_OD2.1mm, F.Cu at (187.1, 127.5)
- added J2: Conn_01x02, Connector_Wire:SolderWire-1.5sqmm_1x02_P6mm_D1.7mm_OD3mm, F.Cu at (199.6, 93.1)
- added J5: Conn_01x06, Connector_Wire:SolderWire-0.5sqmm_1x06_P4.6mm_D0.9mm_OD2.1mm, F.Cu at (182.8, 102.8)
- added J6: Conn_01x02, Connector_Wire:SolderWire-0.5sqmm_1x02_P4.6mm_D0.9mm_OD2.1mm, F.Cu at (186.1, 93.7)
- added J7: Conn_01x04, Connector_PinHeader_2.54mm:PinHeader_1x04_P2.54mm_Vertical, F.Cu at (195.2, 122.8)
- added J8: Conn_01x02, Connector_Wire:SolderWire-0.5sqmm_1x02_P4.6mm_D0.9mm_OD2.1mm, F.Cu at (182.4, 93.6)
- added JP1: Jumper_2_Open, Jumper:SolderJumper-2_P1.3mm_Open_Pad1.0x1.5mm, F.Cu at (133.7, 61.6)
- added JP2: Jumper_2_Open, Jumper:SolderJumper-2_P1.3mm_Open_Pad1.0x1.5mm, F.Cu at (133.7, 65.2)
- added L1: 3.9uH, Inductor:IND_TFM252012ALMA1R0MTAA_TDK, F.Cu at (207.2, 121.8)
- added LED1: XZM2CRKM2DGFBB45SCCB, RGBLED:PLCC4_3p5x2p8_SLD, F.Cu at (200.8, 122.8)
- added MOSFET1: TPC8132_LQS, Package_SO:SOIC-8_3.9x4.9mm_P1.27mm, F.Cu at (209.4, 108.8)
- added Q1: BSS138, Package_TO_SOT_SMD:SOT-23, F.Cu at (140.4, 51.7)
- added Q2: AO3401A, Package_TO_SOT_SMD:SOT-23, F.Cu at (140.4, 56.2)
- added Q3: BSS138, Package_TO_SOT_SMD:SOT-23, F.Cu at (140.4, 60.6)
- added Q4: AO3401A, Package_TO_SOT_SMD:SOT-23, F.Cu at (140.4, 65.1)
- added Q5: BSS138, Package_TO_SOT_SMD:SOT-23, F.Cu at (140.4, 69.5)
- added Q6: AO3401A, Package_TO_SOT_SMD:SOT-23, F.Cu at (140.4, 74.0)
- added R10: 5.5k, Resistor_SMD:R_0603_1608Metric_Pad0.98x0.95mm_HandSolder, F.Cu at (109.3, 55.8)
- added R11: 330, Resistor_SMD:R_0603_1608Metric_Pad0.98x0.95mm_HandSolder, F.Cu at (109.3, 58.3)
- added R12: 120, Resistor_SMD:R_0603_1608Metric_Pad0.98x0.95mm_HandSolder, F.Cu at (109.3, 60.8)
- added R13: 5k, Resistor_SMD:R_0603_1608Metric_Pad0.98x0.95mm_HandSolder, F.Cu at (145.0, 50.7)
- added R14: 10k, Resistor_SMD:R_0603_1608Metric_Pad0.98x0.95mm_HandSolder, F.Cu at (145.0, 53.3)
- added R15: 820, Resistor_SMD:R_0603_1608Metric_Pad0.98x0.95mm_HandSolder, F.Cu at (145.0, 55.8)
- added R16: 5k, Resistor_SMD:R_0603_1608Metric_Pad0.98x0.95mm_HandSolder, F.Cu at (145.0, 58.3)
- added R17: 10k, Resistor_SMD:R_0603_1608Metric_Pad0.98x0.95mm_HandSolder, F.Cu at (149.4, 50.7)
- added R18: 820, Resistor_SMD:R_0603_1608Metric_Pad0.98x0.95mm_HandSolder, F.Cu at (149.4, 53.3)
- added R19: 5k, Resistor_SMD:R_0603_1608Metric_Pad0.98x0.95mm_HandSolder, F.Cu at (149.4, 55.8)
- added R20: 10k, Resistor_SMD:R_0603_1608Metric_Pad0.98x0.95mm_HandSolder, F.Cu at (149.4, 58.3)
- added R21: 510, Resistor_SMD:R_0603_1608Metric_Pad0.98x0.95mm_HandSolder, F.Cu at (153.7, 50.7)
- added R22: 1k, Resistor_SMD:R_0603_1608Metric_Pad0.98x0.95mm_HandSolder, F.Cu at (153.7, 53.3)
- added R23: 1k, Resistor_SMD:R_0603_1608Metric_Pad0.98x0.95mm_HandSolder, F.Cu at (153.7, 55.8)
- added R24: 1k, Resistor_SMD:R_0603_1608Metric_Pad0.98x0.95mm_HandSolder, F.Cu at (153.7, 58.3)
- added R3: 1k, Resistor_SMD:R_0603_1608Metric_Pad0.98x0.95mm_HandSolder, F.Cu at (109.3, 53.3)
- added TP1: TestPoint, TestPoint:TestPoint_Pad_D1.5mm, F.Cu at (201.0, 127.6)
- added U1: STM32F072C8Tx, Package_QFP:LQFP-48_7x7mm_P0.5mm, F.Cu at (192.8, 112.9)
- added U3: SN65HVD232, Package_SO:SOIC-8_3.9x4.9mm_P1.27mm, F.Cu at (194.6, 99.0)
- added U4: AP63203WU, Package_TO_SOT_SMD:TSOT-23-6, F.Cu at (207.6, 115.1)
Routing:
- net +3.3V: track 0.00 -> 16.2 mm
Other:
- board outline added: 51.7 x 49.5 mm
- copper layers 0 -> 2

Commit message: round and tiny board
Parts:
- moved H2 14.4 mm to (211.3, 87.5)
- moved H1 3.66 mm to (180.8, 87.5)
Other:
- board size 51.7 x 49.5 mm -> 37.7 x 46 mm
Changed lines of the file:
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@@
 	(footprint "MountingHole:MountingHole_3.2mm_M3_Pad"
 		(layer "F.Cu")
-		(at 225.298 83.8454)
+		(at 211.35 87.5)
 		(descr "Mounting Hole 3.2mm, M3, generated by kicad-footprint-generator mountinghole.py")
 		(tags "mountinghole M3")
@@
 	(footprint "MountingHole:MountingHole_3.2mm_M3_Pad"
 		(layer "F.Cu")
-		(at 180.6194 83.8454)
+		(at 180.8 87.5)
 		(descr "Mounting Hole 3.2mm, M3, generated by kicad-footprint-generator mountinghole.py")
 		(tags "mountinghole M3")
@@
 	)
 	(gr_rect
-		(start 177.2412 80.4164)
-		(end 228.9048 129.9464)
+		(start 177.2412 83.9)
+		(end 214.95 129.9464)
+		(radius 3.81)
 		(stroke
 			(width 0.05)
-			(type default)
+			(type solid)
 		)
 		(fill no)
